File: hardware/keyswitch_proto_panel.brd (EAGLE design)
At the start: 209.6 x 149.9 mm, 10 parts

Commit message: Handle key matrix presses + handle add event key press
Parts:
- removed U$11, U$12, U$15, U$16, U$7: (no value), mechanical:STANDOFF/3.0
- removed U$14: (no value), mechanical:PIGATRON-LOGO
- added U$1: (no value), mechanical:STANDOFF/3.0
- moved U$2 99.2 mm to (185.3, 58.7)
- moved U$18 12.7 mm to (185.3, 11.7)
- moved U$17 12.2 mm to (26.9, 11.9)
- moved U$13 7.62 mm to (105.4, 11.4), flipped to the bottom
Other:
- board size 209.6 x 149.9 mm -> 166.4 x 54.6 mm
- board text added: "CUT OUT"
- board text removed: "SEQUENCE"
