File: hardware/sequence_panel.brd (EAGLE design)
At the start: 209.6 x 149.9 mm, 10 parts

Commit message: Added source for seperate led matrix driver using atmega328p
Parts:
- added U$1, U$10, U$3, U$4, U$5, U$6, U$8, U$9: (no value), mechanical:STANDOFF/3.0
- added U$19, U$20, U$21, U$22, U$23, U$29, U$30, U$31: HEADER/MALE/01, connectors:HEADER/MALE/01
- moved U$14 141.6 mm to (105.1, 11.4)
- moved U$16 7.73 mm to (54.2, 70.3)
- moved U$13 7.73 mm to (106.7, 11.4)
- moved U$15 1.91 mm to (94.2, 70.3)
- moved U$2 1.91 mm to (94.2, 102.1)
- moved U$7 1.27 mm to (54.2, 102.1)
Connections:
- new net N$1: U$19.1, U$20.1
- new net N$2: U$21.1, U$22.1
- new net N$3: U$23.1, U$29.1
- new net N$4: U$30.1, U$31.1
Routing:
- net N$4: track 0.00 -> 96.7 mm
- net N$3: track 0.00 -> 95.4 mm
- net N$2: track 0.00 -> 5.08 mm
- net N$1: track 0.00 -> 5.08 mm
Other:
- outline, holes or cut-outs redrawn
- board text added: "?"
- board text added: "JLCJLCJLCJLC"
