File: hardware/sequence_panel.sch (EAGLE design)
At the start: 0 parts

Commit message: Added source for seperate led matrix driver using atmega328p
Parts:
- added U$19, U$20, U$21, U$22, U$23, U$29, U$30, U$31: HEADER/MALE/01, connectors:HEADER/MALE/01
Connections:
- new net N$1: U$19.3, U$20.3
- new net N$2: U$21.3, U$22.3
- new net N$3: U$23.3, U$29.3
- new net N$4: U$30.3, U$31.3
Changed lines of the file:
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@@
 </classes>
 <parts>
+<part name="U$19" library="connectors" deviceset="HEADER/MALE/01" device=""/>
+<part name="U$20" library="connectors" deviceset="HEADER/MALE/01" device=""/>
+<part name="U$21" library="connectors" deviceset="HEADER/MALE/01" device=""/>
+<part name="U$22" library="connectors" deviceset="HEADER/MALE/01" device=""/>
+<part name="U$23" library="connectors" deviceset="HEADER/MALE/01" device=""/>
+<part name="U$29" library="connectors" deviceset="HEADER/MALE/01" device=""/>
+<part name="U$30" library="connectors" deviceset="HEADER/MALE/01" device=""/>
+<part name="U$31" library="connectors" deviceset="HEADER/MALE/01" device=""/>
 </parts>
 <sheets>
@@
 </plain>
 <instances>
+<instance part="U$19" gate="HEADER" x="20.32" y="71.12" smashed="yes">
+<attribute name="NAME" x="6.604" y="70.104" size="1.778" layer="96"/>
+</instance>
+<instance part="U$20" gate="HEADER" x="25.4" y="71.12" smashed="yes" rot="R180">
+<attribute name="NAME" x="39.116" y="72.136" size="1.778" layer="96" rot="R180"/>
+</instance>
+<instance part="U$21" gate="HEADER" x="20.32" y="66.04" smashed="yes">
+<attribute name="NAME" x="6.604" y="65.024" size="1.778" layer="96"/>
+</instance>
+<instance part="U$22" gate="HEADER" x="25.4" y="66.04" smashed="yes" rot="R180">
+<attribute name="NAME" x="39.116" y="67.056" size="1.778" layer="96" rot="R180"/>
+</instance>
+<instance part="U$23" gate="HEADER" x="20.32" y="60.96" smashed="yes">
+<attribute name="NAME" x="6.604" y="59.944" size="1.778" layer="96"/>
+</instance>
+<instance part="U$29" gate="HEADER" x="25.4" y="60.96" smashed="yes" rot="R180">
+<attribute name="NAME" x="39.116" y="61.976" size="1.778" layer="96" rot="R180"/>
+</instance>
+<instance part="U$30" gate="HEADER" x="20.32" y="55.88" smashed="yes">
+<attribute name="NAME" x="6.604" y="54.864" size="1.778" layer="96"/>
+</instance>
+<instance part="U$31" gate="HEADER" x="25.4" y="55.88" smashed="yes" rot="R180">
+<attribute name="NAME" x="39.116" y="56.896" size="1.778" layer="96" rot="R180"/>
+</instance>
 </instances>
 <busses>
 </busses>
 <nets>
+<net name="N$1" class="0">
+<segment>
+<pinref part="U$19" gate="HEADER" pin="3"/>
+<pinref part="U$20" gate="HEADER" pin="3"/>
+</segment>
+</net>
+<net name="N$2" class="0">
+<segment>
+<pinref part="U$21" gate="HEADER" pin="3"/>
+<pinref part="U$22" gate="HEADER" pin="3"/>
+</segment>
+</net>
+<net name="N$3" class="0">
+<segment>
+<pinref part="U$23" gate="HEADER" pin="3"/>
+<pinref part="U$29" gate="HEADER" pin="3"/>
+</segment>
+</net>
+<net name="N$4" class="0">
+<segment>
+<pinref part="U$30" gate="HEADER" pin="3"/>
+<pinref part="U$31" gate="HEADER" pin="3"/>
+</segment>
+</net>
 </nets>
 </sheet>
